Commit message: Complete project implementation with comprehensive report and all figures
- Fixed joint limits in robot URDF (realistic ABB IRB1600 specifications)
- Added pause prompts in robot_simulation.m for manual screenshot capture
- Fixed generate_media_online.m (removed blocking calls, added inline functions)
- Generated all 8 required figures (300 DPI, print quality)
- Created comprehensive final report (12,500+ words, 45 pages)
- Generated PDF (FINAL_REPORT.pdf) and PowerPoint (FINAL_PRESENTATION.pptx)
- Added automation scripts: generate_pdf.ps1, verify_media.ps1, list_upload_files.ps1
- Complete documentation: MATLAB Online guides, execution instructions, media guides
- All figures organized in figures/ directory (1.18 MB total)
- Ready for academic submission with professional quality deliverables

File: robot/test.urdf (robot description, URDF)
Before this commit: robot example_robot, 20 links, 19 joints
Joints:
- joint q1: limit lower=-1.57 upper=1.57 effort=10 velocity=3 -> lower=-3.14159 upper=3.14159 effort=10 velocity=3
- joint q2: limit lower=-1.57 upper=1.57 effort=10 velocity=3 -> lower=-1.74533 upper=2.26893 effort=10 velocity=3
- joint q3: limit lower=-1.57 upper=1.57 effort=10 velocity=3 -> lower=-3.14159 upper=1.22173 effort=10 velocity=3
- joint q4: limit lower=-1.57 upper=1.57 effort=10 velocity=3 -> lower=-6.98132 upper=6.98132 effort=10 velocity=3
- joint q5: limit lower=-1.57 upper=1.57 effort=10 velocity=3 -> lower=-2.0944 upper=2.0944 effort=10 velocity=3
- joint q6: limit lower=-1.57 upper=1.57 effort=10 velocity=3 -> lower=-6.98132 upper=6.98132 effort=10 velocity=3
